File: compiled ballin balloon/compiled ballin balloon.kicad_sch (KiCad schematic)
At the start: 0 parts

Commit message: Version 1.0 of Compiled PCB
Other:
- removed sheet Communication
- removed sheet Connectors
- removed sheet Control
- removed sheet IMU
- removed sheet Power
- removed sheet SD card reader
- removed sheet gps
- added sheet Inside (compiled_inside.kicad_sch)
- added sheet Outside (compiled_outside.kicad_sch)
- company: (none) -> SSI Balloons
- title: (none) -> ballin balloon bayload
