File: compiled ballin balloon/compiled_inside.kicad_sch (KiCad schematic)
At the start: 93 parts, among them IC1 CP2104, IC4 BME680, J3 Molex 0510211000, J4 Molex 0510211000, J5 Molex 0532611071, Q10 BSS138, Q5 mmbt2222, Q7 mmbt2222, SW2 KMR2, U1 AZ1117CH-3.3TRG1, U2 TPS82140, U3 TPS82140, U4 TPS82140, U5 3073, U6 TPS82140, U7 TPS82140, X10 GPS_PA1010D, X5 ESP32_WROOM32_SKINNY, X7 microSD, X8 20329, X9 32.768

Commit message: v1.0 with LTC1628 switcher
Parts:
- removed C10, C22, C25, C5: 3.3nF, Capacitor_SMD:C_0603_1608Metric, symbol Device:C_US
- removed C11, C13: 10µF, Capacitor_SMD:C_0603_1608Metric, symbol Adafruit HUZZAH32 ESP32 Feather-eagle-import:CAP_CERAMIC0805-NOOUTLINE
- removed C12: 1uF, Capacitor_SMD:C_0603_1608Metric, symbol Adafruit HUZZAH32 ESP32 Feather-eagle-import:CAP_CERAMIC0603_NO
- removed C19, C23, C26, C8: 22uF, Capacitor_SMD:C_0603_1608Metric, symbol Device:C_US
- removed C20, C24, C9: 10uF, Capacitor_SMD:C_0603_1608Metric, symbol Device:C_US
- removed C27: C_US, Capacitor_SMD:C_0603_1608Metric, symbol Device:C_US
- removed C7: 10uF, Capacitor_SMD:C_0603_1608Metric, symbol Adafruit HUZZAH32 ESP32 Feather-eagle-import:CAP_CERAMIC0805-NOOUTLINE
- removed D7: MBR120, Diode_SMD:D_SOD-123, symbol Adafruit HUZZAH32 ESP32 Feather-eagle-import:DIODE-SCHOTTKYSOD-123
- removed D9: 1N4148, Diode_SMD:D_SOD-323, symbol Adafruit PA1010D Mini GPS-eagle-import:DIODESOD-323
- removed R11, R14: 124k, Resistor_SMD:R_0603_1608Metric, symbol Device:R_US
- removed R12, R15, R35: 100k, Resistor_SMD:R_0603_1608Metric, symbol Device:R_US
- removed R13, R16: 0.5, Resistor_SMD:R_1206_3216Metric, symbol Device:R_US
- removed R62: 10k, Resistor_SMD:R_0603_1608Metric, symbol Device:R_US
- removed U1: AZ1117CH-3.3TRG1, Package_TO_SOT_SMD:SOT-223, symbol AZ1117CH-3.3TRG1:AZ1117CH-3.3TRG1
- removed U2, U3, U4, U6, U7: TPS82140, Package_LGA:Texas_SIL0008D_MicroSiP-8-1EP_2.8x3mm_P0.65mm_EP1.1x1.9mm_ThermalVias, symbol Regulator_Switching:TPS82140
- removed X10: GPS_PA1010D, ballin footprint library:GPS, symbol Adafruit PA1010D Mini GPS-eagle-import:GPS_PA1010D
- removed X8: 20329, Adafruit HUZZAH32 ESP32 Feather:4UCONN_20329_V2, symbol Adafruit HUZZAH32 ESP32 Feather-eagle-import:USB_MICRO_20329_V2
- added C10: 4.7uF, Capacitor_SMD:C_0603_1608Metric, symbol Device:C_Polarized
- added C11, C30, C38: 0.1uF, Capacitor_SMD:C_0603_1608Metric, symbol Device:C_US
- added C28, C33, C37: 1000pF, Capacitor_SMD:C_0603_1608Metric, symbol Device:C_US
- added C29, C36: 180pF, Capacitor_SMD:C_0603_1608Metric, symbol Device:C_US
- added C31: 0.01uF, Capacitor_SMD:C_0603_1608Metric, symbol Device:C_US
- added C32, C34: 33pF, Capacitor_SMD:C_0603_1608Metric, symbol Device:C_US
- added C35: 1000pf, Capacitor_SMD:C_0603_1608Metric, symbol Device:C_US
- added C5: 33uF, Capacitor_SMD:C_0603_1608Metric, symbol Device:C_Polarized
- added C7: 1uF, Capacitor_SMD:C_0603_1608Metric, symbol Device:C_Polarized
- added C8: 150uF, Capacitor_SMD:C_0603_1608Metric, symbol Device:C_Polarized
- added C9: 180uF, Capacitor_SMD:C_0603_1608Metric, symbol Device:C_Polarized
- added D1, D2, D3, D4, D5: D_Schottky, Diode_SMD:D_SOD-323, symbol Device:D_Schottky
- added D7: LED, LED_SMD:LED_0603_1608Metric, symbol Device:LED
- added FB1: FerriteBead, Inductor_SMD:L_0805_2012Metric, symbol Device:FerriteBead
- added J1: USB_C_Receptacle_USB2.0_16P, symbol Connector:USB_C_Receptacle_USB2.0_16P
- added L1: 6.3uH, symbol Device:L_Ferrite
- added Q1, Q2, Q3, Q4: NMOS, symbol Simulation_SPICE:NMOS
- added R17: Input Pullup value, Resistor_SMD:R_0603_1608Metric, symbol Device:R_US
- added R18: Input Pull up value, Resistor_SMD:R_0603_1608Metric, symbol Device:R_US
- added R19: 105k, Resistor_SMD:R_0603_1608Metric, symbol Device:R_US
- added R20, R23: 20k, Resistor_SMD:R_0603_1608Metric, symbol Device:R_US
- added R21, R22: 15k, Resistor_SMD:R_0603_1608Metric, symbol Device:R_US
- added R24: 63.4k, Resistor_SMD:R_0603_1608Metric, symbol Device:R_US
- added R25: 59k, Resistor_SMD:R_0603_1608Metric, symbol Device:R_US
- added TR1: ADTL2-18, RF_Mini-Circuits:Mini-Circuits_CD542_H2.84mm, symbol Transformer:ADTL2-18
- added U1: 5186, CD-PA1616D_ADA, symbol GPS PA 1616:5186
- added U2: LT1129-3.3_TO220_TO263, symbol Regulator_Linear:LT1129-3.3_TO220_TO263
- added U8: LTC1628IG-TRPBF, ballin footprint library:LTC1628IG, symbol LTC1628IG:LTC1628IG-TRPBF
- C1: value 22uF -> 0.1uF
- C2: value 10uF -> 1uF
- C3: value 3.3nF -> 0.1uF
- C4: value 10uF -> 22uF
- J5: footprint (none) -> ballinBreakoutPrints:CONN_532610001-SD_10_MOL
- R1, R4: value 124k -> 100k
- R10: value 0.5 -> 470; footprint Resistor_SMD:R_1206_3216Metric -> Resistor_SMD:R_0603_1608Metric
- R2: value 100k -> 1M
- R3: value 0.5 -> 0.015; footprint Resistor_SMD:R_1206_3216Metric -> Resistor_SMD:R_0603_1608Metric
- R36, R37, R44, R45: footprint (none) -> Resistor_SMD:R_0603_1608Metric
- R5: value 100k -> 220k
- R6: value 0.5 -> 10; footprint Resistor_SMD:R_1206_3216Metric -> Resistor_SMD:R_0603_1608Metric
- R7: value 124k -> 0.01
- R9: value 100k -> 10k
Connections:
- net +12V: now also R6.2, Q2.1 (D), Q3.1 (D); no longer C2.1
- net +3.3V: now also R7.2, R9.1, C36.2, C37.1, C38.2, C9.1, FB1.1, J1.A4 (VBUS), J1.A9 (VBUS), J1.B4 (VBUS), J1.B9 (VBUS), R17.1, R18.1, R24.2, U8.13 (SENSE2-), U8.15 (RUN/SS2)
- net +5V: now also C28.2, C29.1, C5.2, C8.1, R19.2, U8.22 (EXTVCC), U8.3 (SENSE1-); no longer R10.2, R6.1
- net 3.3V: now also U8.10 (3.3VOUT)
- net A13_I35: no longer X5.7 (I35/A1_7)
- net GND: now also R1.1, R4.1, C10.2, C11.2, C30.1, C31.1, C32.1, C34.1, C38.1, C7.2, C8.2, C9.2, D4.2 (A), D5.2 (A), D7.1 (K), J1.A1 (GND), J1.A12 (GND), J1.B1 (GND), J1.B12 (GND), J1.S1 (SHIELD), Q1.3 (S), Q4.3 (S), R20.1, R21.1, R22.1, R23.1, R25.1, U1.12 (GND), U1.19 (GND), U1.3 (GND), U1.8 (GND), U2.3 (GND), U8.20 (PGND), U8.28 (FLTCPL), U8.9 (SGND); no longer C1.2, C3.2, R2.2, R5.2, R9.2
- net SCL_3V: now also U1.14 (RX1(I2C_SCL))
- net SDA_3V: now also U1.15 (TX1(I2C_SDA))
- net at R4.2, R5.1: now also U2.2 (SENSE)
- net at R10.1: now also D7.2 (A); no longer R4.1
- net at IC1.3 (D+): now also IC1.4 (D-), J1.A6 (D+), J1.A7 (D-), J1.B6 (D+), J1.B7 (D-)
- net at C3.1: now also D2.1 (K), U8.18 (BOOST2)
- net at R2.1: now also R25.2, U8.7 (FCB); no longer R1.2
- net at R7.1: now also C37.2, L1.1, U8.14 (SENSE2+)
- net GPS_PPS: now reaches X5.23 (IO15/A2_3)
- net GPS_PPS: now also U1.13 (1PPS)
- net GPS_RESET: now reaches X5.27 (IO16)
- net GPS_RESET: now also R9.2, U1.2 (NRESET)
- new net: C30.2, U8.1 (RUN/SS1)
- new net: Q3.2 (G), U8.16 (TG2)
- new net: C3.2, D5.1 (K), L1.2, Q3.3 (S), Q4.1 (D), U8.17 (SW2)
- new net: D3.2 (A), TR1.1
- new net: C1.1, D4.1 (K), Q1.1 (D), Q2.3 (S), TR1.3, U8.26 (SW1)
- new net: C28.1, R3.1, TR1.4, TR1.6, U8.2 (SENSE1+)
- new net: C35.1, R22.2
- new net: C34.2, C35.2, U8.11 (ITH2)
- new net: FB1.2, U1.1 (VCC), U1.4 (VBACKUP)
- new net: R10.2, U1.5 (3D-FIX)
- new net: C5.1, D3.1 (K), R2.2, U2.5 (IN)
- new net: J1.A5 (CC1), R17.2
- new net: C29.2, R19.1, R20.2, U8.4 (VOSENSE1)
- new net: Q1.2 (G), U8.23 (BG1)
- new net: C33.1, R21.2
- new net: C7.1, R5.2, U2.1 (OUT)
- new net: C36.1, R23.2, R24.1, U8.12 (VOSENSE2)
- new net: C10.1, C2.1, D1.2 (A), D2.2 (A), U8.21 (INTVCC)
- new net: Q4.2 (G), U8.19 (BG2)
- new net: C1.2, D1.1 (K), U8.25 (BOOST1)
- new net: C31.2, U8.6 (STBYMD)
- new net: C11.1, R6.1, U8.24 (VIN)
- new net: Q2.2 (G), U8.27 (TG1)
- new net: C32.2, C33.2, U8.8 (ITH1)
- new net: J1.B5 (CC2), R18.2
- new net A13_135: X5.7 (I35/A1_7)
- new net INTVcc: U8.5 (FREQSET)
- new net ON/OFF: U2.4 (~{SHDN})
- new net VPULL-UP: R1.2
- no-connect marks 33 -> 31
Other:
- note added: "BME SENSOR"
- note added: "DC-DC Switcher 12v-5v-3.3v"
- note added: "Do we want to supply Vbackup with its own battery?"
- note added: "GPS"
- note added: "IMU"
- note added: "SD CARD READER"
- note added: "U2 and T1 are incorrect, I couldn't find the right part so I just picked something with the correct connections"
- note added: "We can connect an antenna if we want. Chip autodetects antenna when there is current draw from EX_ANT"
- note removed: "12V-5V thingy majig"
- note removed: "5V-3.3V regulator"
- note removed: "POWER AND FILTERING"
- company: SSI Balons -> SSI Balloons
- moved on the sheet: C14, C15, C16, C17, C18, C21, D6, D8, H3, H4, IC1A, IC1B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

Commit message: esp32-s3-wroom1u version
Parts:
- removed C5: 33uF, Capacitor_SMD:C_0603_1608Metric, symbol Device:C_Polarized
- removed C7: 1uF, Capacitor_SMD:C_0603_1608Metric, symbol Device:C_Polarized
- removed D3: D_Schottky, Diode_SMD:D_SOD-323, symbol Device:D_Schottky
- removed R25: 59k, Resistor_SMD:R_0603_1608Metric, symbol Device:R_US
- removed R3: 0.015, Resistor_SMD:R_0603_1608Metric, symbol Device:R_US
- removed R4: 100k, Resistor_SMD:R_0603_1608Metric, symbol Device:R_US
- removed R5: 220k, Resistor_SMD:R_0603_1608Metric, symbol Device:R_US
- removed TR1: ADTL2-18, RF_Mini-Circuits:Mini-Circuits_CD542_H2.84mm, symbol Transformer:ADTL2-18
- removed U2: LT1129-3.3_TO220_TO263, symbol Regulator_Linear:LT1129-3.3_TO220_TO263
- added L2: 8uH, symbol Device:L_Ferrite
- added U2: ESP32-S3-WROOM-1U-N4, ballin footprint library:SP32-S3-WROOM-1U-N4, symbol compilled symbol:ESP32-S3-WROOM-1U-N4
- C1, C11, C2, C28, C3, C30, C31, C32, C34, C37, C38, C4: symbol Device:C_US -> Device:C
- C14: symbol Adafruit SDIO microSD-eagle-import:CAP_CERAMIC0805-NOOUTLINE -> Device:C
- C15: symbol Adafruit SDIO microSD-eagle-import:CAP_CERAMIC0603_NO -> Device:C
- C17, C18, C21: symbol Adafruit BNO055 STEMMA QT-eagle-import:microbuilder_CAP_CERAMIC0603_NO -> Device:C
- C29, C36: value 180pF -> 27pF; symbol Device:C_US -> Device:C
- C33: value 1000pF -> 220pF; symbol Device:C_US -> Device:C
- C35: value 1000pf -> 220pF; symbol Device:C_US -> Device:C
- C8: value 150uF -> 47uF
- C9: value 180uF -> 56uF
- L1: value 6.3uH -> 8uH
- R2: value 1M -> 0.015; footprint Resistor_SMD:R_0603_1608Metric -> (none)
- R7: value 0.01 -> 0.015
- U1: footprint CD-PA1616D_ADA -> ballin footprint library:GPS PA1616
Connections:
- net +3.3V: no longer C38.2, U8.15 (RUN/SS2)
- net +5V: now also R2.2
- net 3.3V: now also U8.7 (FCB)
- net at C1.1, D4.1 (K), Q1.1 (D)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: now also L2.2
- net at C28.1, U8.2 (SENSE1+): now also R2.1, L2.1
- net at C35.1, R22.2: now also C34.2
- net at C35.2, U8.11 (ITH2): no longer C34.2
- net at C33.1, R21.2: now also C32.2
- net at C33.2, U8.8 (ITH1): no longer C32.2
- net +12V renamed VBATT
- new net: C38.2, U8.15 (RUN/SS2)
- no-connect marks 31 -> 42
Other:
- note added: "3A; 4A Peak"
- note added: "5.2V to 28V"
- note added: "Connected"
- note added: "DC-DC Switcher 5v and 3.3v output"
- note removed: "DC-DC Switcher 12v-5v-3.3v"
- note removed: "U2 and T1 are incorrect, I couldn't find the right part so I just picked something with the correct connections"
- moved on the sheet: C1, C10, C11, C2, C28, C29, C3, C30, C31, C32, C33, C34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
