File: ballin balloon bayload.kicad_pcb (KiCad board)
At the start: 4 copper layers, 73 x 86 mm, 13 parts, among them J1 Molex 0510211000, J2 Molex 0532611071, J3 Molex 0510211000, J4 Conn_01x06_Pin, J5 Conn_01x06_Pin, U1 MICROSD_SPI_OR_SDIO_CARD, U2 3073, U3 2472

Commit message: updated pcb layout
Parts:
- H1, H2: footprint MountingHole:MountingHole_3.2mm_M3 -> MountingHole:MountingHole_2.5mm
- moved A1 121.2 mm to (190.2, 71.2), turned to -90 degrees
- moved R1 113.1 mm to (162.5, 63.5), turned to -90 degrees
- moved R2 106.7 mm to (148.5, 63.5), turned to -90 degrees
- moved H1 79.8 mm to (98.9, 77.1), turned to -90 degrees
- moved J5 76.8 mm to (200.3, 113.2), turned to -90 degrees
- moved U3 61.5 mm to (155.4, 117.2), turned to 90 degrees
- moved H2 49.8 mm to (98.9, 118.8), turned to -90 degrees
- moved J4 49.2 mm to (174.5, 119.5), turned to 90 degrees
- moved J1 36.2 mm to (80.5, 116.0), turned to 180 degrees
- moved U2 32.8 mm to (122.4, 78.8), turned to 90 degrees
- moved J2 25.3 mm to (74.3, 137.5)
- moved J3 25.2 mm to (80.2, 132.5), turned to 180 degrees
- moved U1 22.5 mm to (124.8, 118.6), turned to 180 degrees
Other:
- board size 73 x 86 mm -> 170 x 87 mm

Commit message: verifying connections before pcb creation
Parts:
- removed J1, J3: Molex 0510211000, Connector_Molex:Molex_PicoBlade_53047-1010_1x10_P1.25mm_Vertical
- J4, J5: footprint Connector_Molex:Molex_PicoBlade_53047-0610_1x06_P1.25mm_Vertical -> Connector_PinHeader_2.54mm:PinHeader_1x06_P2.54mm_Vertical
- moved J2 14.2 mm to (68.4, 124.6)
Connections:
- J2 pad 1: /inside/RX_MCU -> GND
- J2 pad 10: GND -> /inside/RX_MCU
- J2 pad 3: unconnected-(J2-Pin_3-Pad3) -> +5V
- J2 pad 5: unconnected-(J2-Pin_5-Pad5) -> /inside/TX_MCU
- J2 pad 6: /inside/TX_MCU -> unconnected-(J2-Pin_6-Pad6)
- J2 pad 8: +5V -> unconnected-(J2-Pin_8-Pad8)
- J4 pad 3: unconnected-(J4-Pin_3-Pad3) -> GND
