File: inside.kicad_sch (KiCad schematic)
At the start: 13 parts, among them J1 Molex 0510211000, J2 Molex 0532611071, J3 Molex 0510211000, J4 Conn_01x06_Pin, J5 Conn_01x06_Pin, U1 MICROSD_SPI_OR_SDIO_CARD, U2 3073, U3 2472

Commit message: updated pcb layout
Parts:
- H1, H2: footprint MountingHole:MountingHole_3.2mm_M3 -> MountingHole:MountingHole_2.5mm
Changed lines of the file:
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@@
 			)
 		)
-		(property "Footprint" "MountingHole:MountingHole_3.2mm_M3"
+		(property "Footprint" "MountingHole:MountingHole_2.5mm"
 			(at 33.02 124.46 0)
 			(effects
@@
 			)
 		)
-		(property "Footprint" "MountingHole:MountingHole_3.2mm_M3"
+		(property "Footprint" "MountingHole:MountingHole_2.5mm"
 			(at 33.02 116.84 0)
 			(effects

Commit message: verifying connections before pcb creation
Parts:
- J1, J3: footprint Connector_Molex:Molex_PicoBlade_53047-1010_1x10_P1.25mm_Vertical -> (none)
- J4, J5: footprint Connector_Molex:Molex_PicoBlade_53047-0610_1x06_P1.25mm_Vertical -> Connector_PinHeader_2.54mm:PinHeader_1x06_P2.54mm_Vertical
Connections:
- net +5V: now also J2.3 (Pin_3); no longer J1.8 (Pin_8), J2.8 (Pin_8), J3.8 (Pin_8)
- net GND: now also J2.1 (Pin_1), J3.1 (Pin_1), J4.3 (Pin_3); no longer J2.10 (Pin_10), J3.10 (Pin_10)
- net RX_MCU: now also J2.10 (Pin_10), J3.10 (Pin_10); no longer J2.1 (Pin_1), J3.1 (Pin_1)
- net TX_MCU: now also J2.5 (Pin_5), J3.5 (Pin_5); no longer J2.6 (Pin_6), J3.6 (Pin_6)
- net at J1.2 (Pin_2): now also J3.9 (Pin_9); no longer J3.2 (Pin_2)
- net at J1.3 (Pin_3): now also J3.8 (Pin_8); no longer J3.3 (Pin_3)
- net at J1.4 (Pin_4): now also J3.7 (Pin_7); no longer J3.4 (Pin_4)
- net at J1.5 (Pin_5): now also J3.6 (Pin_6); no longer J3.5 (Pin_5)
- net at J1.7 (Pin_7): now also J3.4 (Pin_4); no longer J3.7 (Pin_7)
- net at J1.9 (Pin_9): now also J3.2 (Pin_2); no longer J3.9 (Pin_9)
- new net 5V: J1.8 (Pin_8), J3.3 (Pin_3)
- no-connect marks 26 -> 25
Other:
- note added: "DELETE ONCE SEEN: wrong footprint, edited to be normal 2.5 pins"
- moved on the sheet: J1, J3
