File: _autosave-ballin balloon bayload.kicad_pcb (KiCad board)
At the start: 4 copper layers, 108.5 x 86 mm, 15 parts, among them J2 Molex 0532611071, J4 Conn_01x06_Pin, J5 Conn_01x06_Pin, U1 MICROSD_SPI_OR_SDIO_CARD, U2 3073, U3 2472

Commit message: small tweaks
Parts:
- R1, R2: footprint Resistor_SMD:R_0603_1608Metric -> Resistor_THT:R_Axial_DIN0204_L3.6mm_D1.6mm_P5.08mm_Horizontal
- moved R2 12.3 mm to (109.0, 111.5), turned to -90 degrees
- moved R1 9.55 mm to (108.0, 125.5), turned to 90 degrees
- moved X1 0.60 mm to (43.6, 136.0)
